File: hw/home-media-converter.kicad_pcb (KiCad board)
At the start: 4 copper layers, 79.6 x 54 mm, 148 parts, among them J2 Conn_01x04_Male, J3 Conn_01x03, J4 Conn_01x03, J5 Conn_01x03, J6 RJ45_LED_Shielded, J7 USB_B, SW1 SW_Push, U1 KSZ9131RNXC-TR, U2 STM32F030F4Px, U3 DP83TG720RWRHATQ1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

Commit message: Bigger components on MDI
Parts:
- C16: footprint Capacitor_SMD:C_0402_1005Metric -> Capacitor_SMD:C_1206_3216Metric
- R38: footprint Resistor_SMD:R_0402_1005Metric -> Resistor_SMD:R_0805_2012Metric
- moved C16 1.90 mm to (110.8, 135.4), turned to 90 degrees
- moved R38 0.80 mm to (110.8, 144.0)
Routing:
- net GND: track 60.8 -> 59.3 mm, vias 100 -> 103
- net Net-(C16-Pad1): track 6.31 -> 7.61 mm
