File: hw/power.kicad_sch (KiCad schematic)
At the start: 66 parts, among them J7 USB_B, U1 KSZ9131RNXC-TR, U3 DP83TG720RWRHATQ1, U4 AP63203WU, U5 TPS62A01ADRLR, U6 TPS784105QWDRBRQ1, U7 TPS62A01ADRLR

Commit message: Set missing part values, create BOM
Parts:
- FB2, FB3: value FerriteBead -> BLM18PG121SN1D
- FB4, FB6: value FerriteBead -> BLM18KG601SH1
- FB5: value FerriteBead -> BLM18HE102SN1
Changed lines of the file:
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@@
       (effects (font (size 1.27 1.27)) (justify right))
     )
-    (property "Value" "FerriteBead" (at 61.8236 55.093 0)
+    (property "Value" "BLM18PG121SN1D" (at 61.8236 55.093 0)
       (effects (font (size 1.27 1.27)) (justify right))
     )
@@
       (effects (font (size 1.27 1.27)))
     )
-    (property "Value" "FerriteBead" (at 213.3092 60.9655 90)
+    (property "Value" "BLM18KG601SH1" (at 213.3092 60.9655 90)
       (effects (font (size 1.27 1.27)))
     )
@@
       (effects (font (size 1.27 1.27)) (justify left))
     )
-    (property "Value" "FerriteBead" (at 84.6836 28.3214 0)
+    (property "Value" "BLM18PG121SN1D" (at 84.6836 28.3214 0)
       (effects (font (size 1.27 1.27)) (justify left))
     )
@@
       (effects (font (size 1.27 1.27)))
     )
-    (property "Value" "FerriteBead" (at 213.3092 41.9155 90)
+    (property "Value" "BLM18KG601SH1" (at 213.3092 41.9155 90)
       (effects (font (size 1.27 1.27)))
     )
@@
       (effects (font (size 1.27 1.27)))
     )
-    (property "Value" "FerriteBead" (at 213.3092 49.5355 90)
-      (effects (font (size 1.27 1.27)))
-    )
+    (property "Value" "BLM18HE102SN1" (at 213.3092 49.5355 90)
+      (effects (font (size 1.27 1.27)))
+    )
