File: hw/pcb/power.kicad_sch (KiCad schematic)
At the start: 66 parts, among them J7 USB_B, U1 KSZ9131RNXC-TR, U3 DP83TG720RWRHATQ1, U4 AP63203WU, U5 TPS62A01ADRLR, U6 TPS784105QWDRBRQ1, U7 TPS62A01ADRLR

Commit message: Fix missing part numbers and BOM
Parts:
- F1: value Fuse -> 2A5
- FB1: value FerriteBead -> BLM18PG121SN1D
Changed lines of the file:
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@@
       (effects (font (size 1.27 1.27)))
     )
-    (property "Value" "Fuse" (at 36.83 109.8351 90)
+    (property "Value" "2A5" (at 36.83 109.8351 90)
       (effects (font (size 1.27 1.27)))
     )
@@
       (effects (font (size 1.27 1.27)))
     )
-    (property "Value" "FerriteBead" (at 44.3992 107.9555 90)
+    (property "Value" "BLM18PG121SN1D" (at 44.3992 107.9555 90)
       (effects (font (size 1.27 1.27)))
     )
